File: ad74416h_power_interface_module/ad74416h_power_interface_module.kicad_pcb (KiCad board)
At the start: 4 copper layers, 55.9 x 40.6 mm, 123 parts, among them J1 FW-33-03-G-D-085-155, T1 ZA9644-AED, U1 MAX17227JATA+, U2 MAX17614ATP+, U3 MAX17570FATA+, U4 ADP1031ACPZ-3-R7, U5 ADUM340E0BRQZ, U6 ADUM340E0BRQZ, U7 ADUM1252AUA+

Commit message: backup
Parts:
- moved TP20 3.81 mm to (152.4, 78.8)
- moved TP23 3.81 mm to (148.5, 78.8)
- moved C17 3.56 mm to (151.2, 103.6)
- moved C23 3.56 mm to (151.2, 113.4)
- moved U6 3.56 mm to (153.4, 108.5)
- moved C16 2.54 mm to (145.4, 103.6)
- moved C22 2.54 mm to (145.4, 113.4)
- moved U5 2.54 mm to (147.6, 108.5)
- moved TP43 1.27 mm to (147.2, 119.4)
- moved TP44 1.27 mm to (148.4, 119.4)
- moved TP46 1.27 mm to (151.0, 119.4)
- moved TP45 1.27 mm to (149.7, 119.4)
Connections:
- J1 pad 39: /5V0 -> /-15V0
- J1 pad 40: /5V0 -> /-15V0
- J1 pad 45: /-15V0 -> /5V0
- J1 pad 46: /-15V0 -> /5V0
Routing:
- net /1B2: track 36.6 -> 34.1 mm
- net /1B1: track 36.1 -> 33.7 mm
- net /2B3: track 35.3 -> 33.1 mm
- net /2B4: track 35.8 -> 33.6 mm
- net /SDO: track 40.4 -> 38.3 mm
- net /SDI: track 41.8 -> 39.6 mm
- net /~{SYNC}: track 42.1 -> 39.9 mm
- net /SCLK: track 40.8 -> 38.7 mm
- net /1B3: track 36.3 -> 34.4 mm
- net /1B4: track 36.6 -> 34.7 mm
- net /1B1_ISO: track 6.99 -> 8.08 mm
- net /2B4_ISO: track 8.12 -> 7.06 mm
- net /2B2: track 33.6 -> 32.6 mm
- net /2B1: track 35.4 -> 34.4 mm
- net GNDA: track 0.00 -> 0.76 mm
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- added copper zone on In1.Cu, net /5V0
- removed copper zone on B.Cu, net /5V0

Commit message: backup
Parts:
- moved R21 10.4 mm to (168.1, 115.2), turned to 90 degrees
- moved TP1 10.1 mm to (124.4, 88.9)
- moved TP10 10.1 mm to (135.9, 88.9)
- moved TP11 10.1 mm to (137.1, 88.9)
- moved TP12 10.1 mm to (138.4, 88.9)
- moved TP13 10.1 mm to (139.7, 88.9)
- moved TP14 10.1 mm to (141.0, 88.9)
- moved TP15 10.1 mm to (142.2, 88.9)
- moved TP16 10.1 mm to (143.5, 88.9)
- moved TP17 10.1 mm to (144.8, 88.9)
- moved TP18 10.1 mm to (146.0, 88.9)
- moved TP19 10.1 mm to (147.3, 88.9)
- moved TP2 10.1 mm to (125.7, 88.9)
- moved TP20 10.1 mm to (152.4, 88.9)
- moved TP21 10.1 mm to (149.8, 88.9)
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Routing:
- net /SDA: track 33.4 -> 42.0 mm
- net /SCL: track 34.0 -> 40.4 mm
- net /2B1: track 34.4 -> 30.3 mm
- net /SDI: track 39.6 -> 36.6 mm
- net /~{SYNC}: track 39.9 -> 36.9 mm
- net /SCLK: track 38.7 -> 35.7 mm
- net /SDO: track 38.3 -> 35.3 mm
- net /SDA_ISO: track 6.17 -> 8.96 mm
- net /1B1: track 33.7 -> 31.2 mm
- net /1B2: track 34.1 -> 31.7 mm
- net /2B2: track 32.6 -> 30.3 mm
- net /2B3: track 33.1 -> 30.9 mm
- net /1B3: track 34.4 -> 32.2 mm
- net /2B4: track 33.6 -> 31.7 mm
- net /3V3: track 31.2 -> 29.3 mm
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
Commit message: backup
Parts:
- added MB5: mouse-bite-50mil-1750mil, mouse_bite_footprints:mouse-bite-50mil-1750mil, F.Cu at (144.8, 88.3)
Other:
- outline, holes or cut-outs redrawn

Commit message: backup
Parts:
- added J2: TBP02R1-381-02BE, connector_footprints:TBP02R1-381-02BE, F.Cu at (122.5, 122.6)
- added J3: FW-17-03-G-D-085-155, connector_footprints:FW-17-03-G-D-085-155, F.Cu at (144.8, 124.5)
- added J4: TBP02R1-381-02BE, connector_footprints:TBP02R1-381-02BE, F.Cu at (167.0, 122.6)
- added MB1: mouse-bite-50mil-200mil, mouse_bite_footprints:mouse-bite-50mil-200mil, F.Cu at (122.5, 120.0)
- added MB2: mouse-bite-50mil-950mil, mouse_bite_footprints:mouse-bite-50mil-950mil, F.Cu at (144.8, 120.0)
- added MB3: mouse-bite-50mil-200mil, mouse_bite_footprints:mouse-bite-50mil-200mil, F.Cu at (167.0, 120.0)
- added TP56: TestPoint, test_point_footprints:TestPoint_THTPad_Castelated, F.Cu at (166.4, 119.4)
- added TP57: TestPoint, test_point_footprints:TestPoint_THTPad_Castelated, F.Cu at (167.6, 119.4)
- L3, L4: value 100 µH -> 100.0 µH
- moved TP34 9.91 mm to (121.9, 119.4)
- moved TP35 9.91 mm to (123.2, 119.4)
- moved TP51 6.10 mm to (154.9, 119.4)
- moved TP52 6.10 mm to (153.7, 119.4)
- moved TP47 4.83 mm to (148.6, 119.4)
- moved TP49 4.83 mm to (151.1, 119.4)
- moved TP48 4.83 mm to (149.8, 119.4)
- moved TP50 4.83 mm to (152.4, 119.4)
- moved TP44 3.56 mm to (144.8, 119.4)
- moved TP45 3.56 mm to (146.0, 119.4)
- moved TP46 3.56 mm to (147.3, 119.4)
- moved TP43 3.56 mm to (143.5, 119.4)
- moved TP38 2.29 mm to (137.1, 119.4)
- moved TP36 2.29 mm to (134.6, 119.4)
- moved TP37 2.29 mm to (135.9, 119.4)
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Routing:
- net /DO_VDD: track 7.12 -> 44.7 mm
- net /SDA_ISO: track 8.96 -> 18.0 mm
- net /SCL_ISO: track 7.16 -> 15.8 mm
- net /1B4_ISO: track 7.24 -> 15.8 mm
- net /2B4_ISO: track 7.00 -> 15.3 mm
- net /1B3_ISO: track 7.50 -> 15.3 mm
- net /2B3_ISO: track 7.27 -> 15.0 mm
- net /SDO_ISO: track 10.6 -> 18.3 mm
- net /SCLK_ISO: track 10.6 -> 18.2 mm
- net /1B2_ISO: track 7.76 -> 15.0 mm
- net /~{SYNC_ISO}: track 11.9 -> 19.1 mm
- net /2B2_ISO: track 7.53 -> 14.8 mm
- net /MVDD: track 17.1 -> 24.2 mm
- net /SDI_ISO: track 10.1 -> 17.1 mm
- net /1B1_ISO: track 8.02 -> 14.8 mm
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Other:
- board size 55.9 x 40.6 mm -> 55.9 x 52.3 mm
