File: ad74416h_power_interface_module/ad74416h_power_interface_module.kicad_pcb (KiCad board)
At the start: 4 copper layers, 55.9 x 52.3 mm, 132 parts, among them J1 FW-33-03-G-D-085-155, J2 TBP02R1-381-02BE, J3 FW-17-03-G-D-085-155, J4 TBP02R1-381-02BE, T1 ZA9644-AED, U1 MAX17227JATA+, U2 MAX17614ATP+, U3 MAX17570FATA+, U4 ADP1031ACPZ-3-R7, U5 ADUM340E0BRQZ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

Commit message: backup
Parts:
- moved J2 12.6 mm to (113.6, 113.7), turned to 90 degrees
- moved J4 12.6 mm to (175.9, 113.7), turned to -90 degrees
- moved MB3 8.98 mm to (173.3, 113.7), turned to -90 degrees
- moved MB1 8.98 mm to (116.2, 113.7), turned to 90 degrees
- moved TP56 8.98 mm to (172.7, 113.0), turned to 180 degrees
- moved TP35 8.13 mm to (116.8, 114.3), turned to 0 degrees
- moved TP34 8.13 mm to (116.8, 113.0), turned to 0 degrees
- moved TP57 7.18 mm to (172.7, 114.3), turned to 180 degrees
Connections:
- net /CLMODE renamed /Power_Supply_and_Digital_Interface/CLMODE
- net /EN renamed /Power_Supply_and_Digital_Interface/EN
- net /FB renamed /Power_Supply_and_Digital_Interface/FB
- net /FB1 renamed /Power_Supply_and_Digital_Interface/FB1
- net /FB3 renamed /Power_Supply_and_Digital_Interface/FB3
- net /LX renamed /Power_Supply_and_Digital_Interface/LX
- net /MAX17227_VIN renamed /Power_Supply_and_Digital_Interface/MAX17227_VIN
- net /MAX17570_VIN renamed /Power_Supply_and_Digital_Interface/MAX17570_VIN
- net /OVLO renamed /Power_Supply_and_Digital_Interface/OVLO
- net /RT/SYNC renamed /Power_Supply_and_Digital_Interface/RT/SYNC
- net /SETI renamed /Power_Supply_and_Digital_Interface/SETI
- net /SLEW renamed /Power_Supply_and_Digital_Interface/SLEW
- net /SW2 renamed /Power_Supply_and_Digital_Interface/SW2
- net /SW3 renamed /Power_Supply_and_Digital_Interface/SW3
- net /SWP renamed /Power_Supply_and_Digital_Interface/SWP
- net /SYNC renamed /Power_Supply_and_Digital_Interface/SYNC
- net /TSTART renamed /Power_Supply_and_Digital_Interface/TSTART
- net /UVLO renamed /Power_Supply_and_Digital_Interface/UVLO
- net /UVOV renamed /Power_Supply_and_Digital_Interface/UVOV
- net /VCC renamed /Power_Supply_and_Digital_Interface/VCC
- net /~{FLAG} renamed /Power_Supply_and_Digital_Interface/~{FLAG}
- J4 pad 1: GNDA -> /DO_VDD
- J4 pad 2: /DO_VDD -> GNDA
Routing:
- net /DO_VDD: track 44.7 -> 38.0 mm
Other:
- board size 55.9 x 52.3 mm -> 79.3 x 50.2 mm

Commit message: backup
Parts:
- moved R23 0.88 mm to (137.1, 112.3)
Routing:
- net /DO_VDD: track 38.0 -> 7.12 mm
- net /SCL: track 40.4 -> 38.1 mm
- net /SDA: track 42.0 -> 40.2 mm
- net /1B2: track 31.7 -> 30.7 mm
- net /~{SYNC}: track 36.9 -> 36.1 mm
- net /SDO: track 35.3 -> 34.5 mm
- net /1B4: track 33.3 -> 32.6 mm
- net /2B2: track 30.3 -> 29.6 mm
- net /SDI: track 36.6 -> 36.0 mm
- net /1B1: track 31.2 -> 30.6 mm
- net /2B1: track 30.3 -> 29.7 mm
- net /1B3: track 32.2 -> 31.6 mm
- net /SCLK: track 35.7 -> 35.1 mm
- net GNDA: vias 98 -> 97
- net /24V0: vias 14 -> 17
- added copper zone on B.Cu, net /24V0
- added copper zone on B.Cu, net /DO_VDD

Commit message: backup
Parts:
- added MB4: mouse-bite-50mil-200mil, mouse_bite_footprints:mouse-bite-50mil-200mil, F.Cu at (125.1, 120.0)
- added MB6: mouse-bite-50mil-200mil, mouse_bite_footprints:mouse-bite-50mil-200mil, F.Cu at (164.4, 120.0)
- added TP53: TestPoint, test_point_footprints:TestPoint_THTPad_Castelated, F.Cu at (165.1, 119.4)
- added TP54: TestPoint, test_point_footprints:TestPoint_THTPad_Castelated, F.Cu at (163.8, 119.4)
- added TP55: TestPoint, test_point_footprints:TestPoint_THTPad_Castelated, F.Cu at (125.7, 119.4)
- added TP58: TestPoint, test_point_footprints:TestPoint_THTPad_Castelated, F.Cu at (124.4, 119.4)
- moved J2 9.55 mm to (113.0, 123.2)
- moved J4 9.55 mm to (176.5, 123.2)
- moved TP35 9.53 mm to (116.8, 123.8)
- moved TP57 9.53 mm to (172.7, 123.8)
- moved MB1 9.52 mm to (116.2, 123.2)
- moved MB3 9.52 mm to (173.3, 123.2)
- moved TP34 9.52 mm to (116.8, 122.6)
- moved TP56 9.52 mm to (172.7, 122.6)
Other:
- board size 79.3 x 50.2 mm -> 80.9 x 50.2 mm
