File: ad74416h_power_interface_module/ad74416h_power_interface_module.kicad_pcb (KiCad board)
At the start: 4 copper layers, 80.9 x 50.2 mm, 138 parts, among them J1 FW-33-03-G-D-085-155, J2 TBP02R1-381-02BE, J3 FW-17-03-G-D-085-155, J4 TBP02R1-381-02BE, T1 ZA9644-AED, U1 MAX17227JATA+, U2 MAX17614ATP+, U3 MAX17570FATA+, U4 ADP1031ACPZ-3-R7, U5 ADUM340E0BRQZ, U6 ADUM340E0BRQZ, U7 ADUM1252AUA+

Commit message: backup
Parts:
- added J5: FW-06-03-G-D-085-155, connector_footprints:FW-06-03-G-D-085-155, F.Cu at (125.1, 124.5)
- added J6: FW-06-03-G-D-085-155, connector_footprints:FW-06-03-G-D-085-155, F.Cu at (164.4, 124.5)
- added TP59: TestPoint, test_point_footprints:TestPoint_THTPad_Castelated, F.Cu at (123.2, 119.4)
- added TP60: TestPoint, test_point_footprints:TestPoint_THTPad_Castelated, F.Cu at (127.0, 119.4)
- added TP61: TestPoint, test_point_footprints:TestPoint_THTPad_Castelated, F.Cu at (116.8, 122.6)
- added TP62: TestPoint, test_point_footprints:TestPoint_THTPad_Castelated, F.Cu at (116.8, 126.4)
- added TP63: TestPoint, test_point_footprints:TestPoint_THTPad_Castelated, F.Cu at (128.3, 119.4)
- added TP64: TestPoint, test_point_footprints:TestPoint_THTPad_Castelated, F.Cu at (121.9, 119.4)
- added TP65: TestPoint, test_point_footprints:TestPoint_THTPad_Castelated, F.Cu at (172.7, 122.6)
- added TP66: TestPoint, test_point_footprints:TestPoint_THTPad_Castelated, F.Cu at (172.7, 126.4)
- added TP67: TestPoint, test_point_footprints:TestPoint_THTPad_Castelated, F.Cu at (162.5, 119.4)
- added TP68: TestPoint, test_point_footprints:TestPoint_THTPad_Castelated, F.Cu at (161.3, 119.4)
- added TP69: TestPoint, test_point_footprints:TestPoint_THTPad_Castelated, F.Cu at (166.4, 119.4)
- added TP70: TestPoint, test_point_footprints:TestPoint_THTPad_Castelated, F.Cu at (167.6, 119.4)
- MB1, MB3: value mouse-bite-50mil-200mil -> mouse-bite-50mil-300mil; footprint mouse_bite_footprints:mouse-bite-50mil-200mil -> mouse_bite_footprints:mouse-bite-50mil-300mil
- MB4, MB6: value mouse-bite-50mil-200mil -> mouse-bite-50mil-400mil; footprint mouse_bite_footprints:mouse-bite-50mil-200mil -> mouse_bite_footprints:mouse-bite-50mil-400mil
- moved MB1 1.27 mm to (116.2, 124.5)
- moved MB3 1.27 mm to (173.3, 124.5)
- moved TP34 1.27 mm to (116.8, 123.8)
- moved TP56 1.27 mm to (172.7, 123.8)
- moved C18 1.27 mm to (168.1, 110.8)
- moved C19 1.27 mm to (166.6, 110.8)
- moved C24 1.27 mm to (158.9, 110.8)
- moved C25 1.27 mm to (157.4, 110.8)
- moved J2 1.27 mm to (113.0, 124.5)
- moved J4 1.27 mm to (176.5, 124.5)
- moved R21 1.27 mm to (168.1, 113.9)
- moved R22 1.27 mm to (166.6, 113.9)
- moved R24 1.27 mm to (158.9, 113.9)
- moved R25 1.27 mm to (157.4, 113.9)
- moved TP35 1.27 mm to (116.8, 125.1)
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Routing:
- net /SCL_ISO: track 15.5 -> 16.7 mm
- net /SDA_ISO: track 17.7 -> 18.9 mm
- net /SCL: track 38.1 -> 37.0 mm
- net /SDA: track 40.2 -> 39.2 mm
Other:
- board size 80.9 x 50.2 mm -> 80.9 x 51.4 mm

Commit message: backup
Parts:
- removed the TP63 at (128.3, 119.4)
- removed the TP64 at (121.9, 119.4)
- removed TP68, TP70: TestPoint, test_point_footprints:TestPoint_THTPad_Castelated
- J3: renamed from J5; value FW-06-03-G-D-085-155 -> FW-04-03-G-D-085-155; footprint connector_footprints:FW-06-03-G-D-085-155 -> connector_footprints:FW-04-03-G-D-085-155
- J5: renamed from J6; value FW-06-03-G-D-085-155 -> FW-04-03-G-D-085-155; footprint connector_footprints:FW-06-03-G-D-085-155 -> connector_footprints:FW-04-03-G-D-085-155
- MB2: renamed from MB4; value mouse-bite-50mil-400mil -> mouse-bite-50mil-300mil; footprint mouse_bite_footprints:mouse-bite-50mil-400mil -> mouse_bite_footprints:mouse-bite-50mil-300mil
- MB4: renamed from MB6; value mouse-bite-50mil-400mil -> mouse-bite-50mil-300mil; footprint mouse_bite_footprints:mouse-bite-50mil-400mil -> mouse_bite_footprints:mouse-bite-50mil-300mil
- moved J2 0.64 mm to (113.0, 125.1)
- moved J3 0.64 mm to (125.1, 125.1)
- moved J4 0.64 mm to (144.8, 125.1)
- moved J5 0.64 mm to (164.4, 125.1)
- moved J6 0.64 mm to (176.5, 125.1)
- moved TP59 0.64 mm to (116.8, 123.2)
- moved TP60 0.64 mm to (172.7, 123.2)
- moved TP65 0.64 mm to (116.8, 127.0)
- moved TP66 0.64 mm to (172.7, 127.0)
- moved MB5 0.63 mm to (116.2, 125.1)
- moved MB6 0.63 mm to (173.3, 125.1)
- moved TP61 0.63 mm to (116.8, 124.5)
- moved TP62 0.63 mm to (172.7, 124.5)
- moved TP63 0.63 mm to (116.8, 125.7)
- moved TP64 0.63 mm to (172.7, 125.7)
- renumbered C12 to C10, C15 to C11, C7 to C12, C8 to C13, C16 to C14, C17 to C15, C13 to C16, C14 to C17, C25 to C18, C24 to C19, C4 to C2, C19 to C20, C18 to C21, C20 to C22, C21 to C23, C22 to C24, C23 to C25, C6 to C3, C5 to C4, C2 to C5, C9 to C6, C3 to C7, C10 to C8, C11 to C9, J3 to J4, J4 to J6, L3 to L2, L4 to L3, L2 to L4, MB5 to MB1, MB2 to MB3, MB1 to MB5, MB3 to MB6, R11 to R10, R4 to R11, R14 to R12, R15 to R13, R16 to R14, R17 to R15, R5 to R16, R13 to R17, R3 to R2, R23 to R21, R25 to R22, R24 to R23, R22 to R24, R21 to R25, R2 to R3, R6 to R4, R7 to R5, R10 to R6, R12 to R7, TP23 to TP20, TP20 to TP23, TP59 to TP34, TP58 to TP35, TP55 to TP36, TP60 to TP37, TP36 to TP38, TP37 to TP39, TP38 to TP40, TP39 to TP41, TP40 to TP42, TP41 to TP43, TP42 to TP44, TP43 to TP45, TP44 to TP46, TP45 to TP47, TP46 to TP48, TP47 to TP49, TP48 to TP50, TP49 to TP51, TP50 to TP52, TP52 to TP53, TP51 to TP54, TP67 to TP55, TP54 to TP56, TP53 to TP57, TP69 to TP58, TP61 to TP59, TP65 to TP60, TP34 to TP61, TP56 to TP62, TP35 to TP63, TP57 to TP64, TP62 to TP65
Connections:
- J3 pad 5: /VINP -> GND
- J3 pad 6: /VINP -> GND
- J5 pad 5: GNDA -> /DO_VDD
- J5 pad 6: GNDA -> /DO_VDD
Routing:
- net /SCLK_ISO: track 17.9 -> 18.6 mm
- net /~{SYNC_ISO}: track 18.7 -> 19.4 mm
- net /SDO_ISO: track 17.9 -> 18.5 mm
- net /SDI_ISO: track 16.9 -> 17.5 mm
- net /SDA_ISO: track 18.9 -> 19.5 mm
- net /SCL_ISO: track 16.7 -> 17.4 mm
- net /PWRGD: track 16.7 -> 17.3 mm
- net /MVDD: track 24.2 -> 24.9 mm
- net /2B4_ISO: track 15.2 -> 15.8 mm
- net /2B3_ISO: track 14.8 -> 15.5 mm
- net /2B2_ISO: track 14.5 -> 15.2 mm
- net /2B1_ISO: track 14.3 -> 14.9 mm
- net /1B4_ISO: track 15.7 -> 16.4 mm
- net /1B3_ISO: track 15.2 -> 15.8 mm
- net /1B2_ISO: track 14.8 -> 15.5 mm
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Other:
- board size 80.9 x 51.4 mm -> 80.9 x 52.1 mm

Commit message: backup
Parts:
- removed MB5, MB6: mouse-bite-50mil-300mil, mouse_bite_footprints:mouse-bite-50mil-300mil
- removed TP59, TP60, TP61, TP62, TP63, TP64, TP65, TP66: TestPoint, test_point_footprints:TestPoint_THTPad_Castelated
- J1: value FW-33-03-G-D-085-155 -> FW-33-03-G-D-150-160; footprint connector_footprints:FW-33-03-G-D-085-155 -> connector_footprints:FW-33-03-G-D-150-160
Other:
- outline, holes or cut-outs redrawn
