File: ad74416h_power_interface_module/Power_Supply_and_Digital_Interface.kicad_sch (KiCad schematic)
At the start: 124 parts, among them T1 ZA9644-AED, U1 MAX17227JATA+, U2 MAX17614ATP+, U3 MAX17570FATA+, U4 ADP1031ACPZ-3-R7, U5 ADUM340E0BRQZ, U6 ADUM340E0BRQZ, U7 ADUM1252AUA+

Commit message: backup
Parts:
- added TP53, TP54, TP55, TP58: TestPoint, test_point_footprints:TestPoint_THTPad_Castelated, symbol UNITED_TEST_POINTS:TestPoint_Castelated_v2
Connections:
- net DO_VDD: now also TP53.1
- net GND: now also TP55.1
- net GNDA: now also TP54.1
- net VINP: now also TP58.1

Commit message: backup
Parts:
- removed TP53, TP54, TP55, TP58: TestPoint, test_point_footprints:TestPoint_THTPad_Castelated, symbol UNITED_TEST_POINTS:TestPoint_Castelated_v2
- added TP61, TP62, TP65, TP66: TestPoint, test_point_footprints:TestPoint_THTPad_Castelated, symbol UNITED_TEST_POINTS:TestPoint_Castelated_v2
Connections:
- net DO_VDD: now also TP65.1
- net GND: now also TP62.1
- net GNDA: now also TP66.1
- net VINP: now also TP61.1

Commit message: backup
Parts:
- renumbered C12 to C10, C15 to C11, C7 to C12, C8 to C13, C16 to C14, C17 to C15, C13 to C16, C14 to C17, C25 to C18, C24 to C19, C4 to C2, C19 to C20, C18 to C21, C20 to C22, C21 to C23, C22 to C24, C23 to C25, C6 to C3, C5 to C4, C2 to C5, C9 to C6, C3 to C7, C10 to C8, C11 to C9, L3 to L2, L4 to L3, L2 to L4, R11 to R10, R4 to R11, R14 to R12, R15 to R13, R16 to R14, R17 to R15, R5 to R16, R13 to R17, R3 to R2, R23 to R21, R25 to R22, R24 to R23, R22 to R24, R21 to R25, R2 to R3, R6 to R4, R7 to R5, R10 to R6, R12 to R7, TP23 to TP20, TP20 to TP23, TP36 to TP38, TP37 to TP39, TP38 to TP40, TP39 to TP41, TP40 to TP42, TP41 to TP43, TP42 to TP44, TP43 to TP45, TP44 to TP46, TP45 to TP47, TP46 to TP48, TP47 to TP49, TP48 to TP50, TP49 to TP51, TP50 to TP52, TP52 to TP53, TP51 to TP54, TP61 to TP59, TP65 to TP60, TP34 to TP61, TP56 to TP62, TP35 to TP63, TP57 to TP64, TP62 to TP65

Commit message: backup
Parts:
- removed TP59, TP60, TP61, TP62, TP63, TP64, TP65, TP66: TestPoint, test_point_footprints:TestPoint_THTPad_Castelated, symbol UNITED_TEST_POINTS:TestPoint_Castelated_v2
