File: ad74416h_power_interface_module/ad74416h_power_interface_module.kicad_sch (KiCad schematic)
At the start: 123 parts, among them J1 FW-33-03-G-D-085-155, T1 ZA9644-AED, U1 MAX17227JATA+, U2 MAX17614ATP+, U3 MAX17570FATA+, U4 ADP1031ACPZ-3-R7, U5 ADUM340E0BRQZ, U6 ADUM340E0BRQZ, U7 ADUM1252AUA+

Commit message: backup
Connections:
- net -15V0: now also J1.39, J1.40; no longer J1.45, J1.46
- net 5V0: now also J1.45, J1.46; no longer J1.39, J1.40
Changed lines of the file:
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@@
 	)
 	(label "5V0"
-		(at 48.26 88.9 0)
+		(at 48.26 96.52 0)
 		(effects
 			(font
@@
 	)
 	(label "-15V0"
-		(at 27.94 96.52 180)
+		(at 27.94 88.9 180)
 		(effects
 			(font
@@
 	)
 	(label "5V0"
-		(at 27.94 88.9 180)
+		(at 27.94 96.52 180)
 		(effects
 			(font
@@
 	)
 	(label "-15V0"
-		(at 48.26 96.52 0)
+		(at 48.26 88.9 0)
 		(effects
 			(font

Commit message: backup
Parts:
- added MB5: mouse-bite-50mil-1750mil, mouse_bite_footprints:mouse-bite-50mil-1750mil, symbol UNITED_MOUSE_BITES_DATA_BASE:mouse-bite-50mil-1750mil
Other:
- moved on the sheet: C1, C10, C11, C12, C13, C14, C15, C16, C17, C18, C19, C20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

Commit message: backup
Parts:
- added J2, J4: TBP02R1-381-02BE, connector_footprints:TBP02R1-381-02BE, symbol CONNECTORS_TBP02R1-381_DATA_BASE:J_TBP02R1-381-02BE
- added J3: FW-17-03-G-D-085-155, connector_footprints:FW-17-03-G-D-085-155, symbol CONNECTORS_FW-xx-03-G-D-085-155_DATA_BASE:J_FW-17-03-G-D-085-155
- added MB1, MB3: mouse-bite-50mil-200mil, mouse_bite_footprints:mouse-bite-50mil-200mil, symbol UNITED_MOUSE_BITES_DATA_BASE:mouse-bite-50mil-200mil
- added MB2: mouse-bite-50mil-950mil, mouse_bite_footprints:mouse-bite-50mil-950mil, symbol UNITED_MOUSE_BITES_DATA_BASE:mouse-bite-50mil-950mil
- added TP56, TP57: TestPoint, test_point_footprints:TestPoint_THTPad_Castelated, symbol UNITED_TEST_POINTS:TestPoint_Castelated_v2
- L3, L4: value 100 µH -> 100.0 µH
Connections:
- net 1B1_ISO: now also J3.29, J3.30
- net 1B2_ISO: now also J3.27, J3.28
- net 1B3_ISO: now also J3.25, J3.26
- net 1B4_ISO: now also J3.23, J3.24
- net 2B1_ISO: now also J3.21, J3.22
- net 2B2_ISO: now also J3.19, J3.20
- net 2B3_ISO: now also J3.17, J3.18
- net 2B4_ISO: now also J3.15, J3.16
- net DO_VDD: now also J4.2, TP56.1
- net GND: now also J2.1
- net GNDA: now also J4.1, TP57.1
- net GNDD: now also J3.3, J3.4
- net MVDD: now also J3.1, J3.2
- net PWRGD: now also J3.5, J3.6
- net SCLK_ISO: now also J3.10, J3.9
- net SCL_ISO: now also J3.33, J3.34
- net SDA_ISO: now also J3.31, J3.32
- net SDI_ISO: now also J3.7, J3.8
- net SDO_ISO: now also J3.11, J3.12
- net VINP: now also J2.2
- net ~{SYNC_ISO}: now also J3.13, J3.14
Other:
- moved on the sheet: TP43, TP44, TP45, TP46, TP47, TP48, TP49, TP50

Commit message: backup
Parts:
- removed C1: 220 nF, capacitor_footprints:C_0402_1005Metric, symbol CAPACITORS_KGM05AR71C_DATA_BASE:C_KGM05AR71C224KH
- removed C10, C5: 10 µF, capacitor_footprints:C_0603_1608Metric, symbol CAPACITORS_C1608X5R1C_DATA_BASE:C_C1608X5R1C106M080AB
- removed C11, C12, C16, C17, C19, C20, C22, C23, C25: 100 nF, capacitor_footprints:C_0402_1005Metric, symbol UNITED_CAPACITORS_DATA_BASE:C_GCM155R71H104KE02D
- removed C13: 1 µF, capacitor_footprints:C_0402_1005Metric, symbol CAPACITORS_C1005X6S1C_DATA_BASE:C_C1005X6S1C105K050BC
- removed C14: 1 µF, capacitor_footprints:C_0805_2012Metric, symbol CAPACITORS_GRJ21BC72A_DATA_BASE:C_GRJ21BC72A105KE11L
- removed C15, C4, C6: 10 µF, capacitor_footprints:C_1206_3216Metric, symbol UNITED_CAPACITORS_DATA_BASE:C_CL31B106KBHNNN#
- removed C18, C24: 1 nF, capacitor_footprints:C_0402_1005Metric, symbol UNITED_CAPACITORS_DATA_BASE:C_GCM155R71H102KA37D
- removed C2: 10 µF, capacitor_footprints:C_1206_3216Metric, symbol CAPACITORS_CL31B_DATA_BASE:C_CL31B106KBHNNN#
- removed C21: 4.7 µF, capacitor_footprints:C_1210_200_3225Metric, symbol UNITED_CAPACITORS_DATA_BASE:C_GCM32DC72A475KE02K
- removed C3, C7: 100 nF, capacitor_footprints:C_0603_1608Metric, symbol CAPACITORS_C1608X7S2A_DATA_BASE:C_C1608X7S2A104K080AB
- removed C8: 220 pF, capacitor_footprints:C_0402_1005Metric, symbol CAPACITORS_CGA2B2NP02A_DATA_BASE:C_CGA2B2NP02A221J050BA
- removed C9: 4.7 µF, capacitor_footprints:C_0603_1608Metric, symbol UNITED_CAPACITORS_DATA_BASE:C_C1608X7S1A475K080AC
- removed D1, D2: 1.8 V, diode_footprints:LED_RED_0402_1005Metric, symbol DIODES_APHHS1005LSECK-J3-PF_DATA_BASE:D_APHHS1005LSECK-J3-PF
- removed D3: 200.0 V, diode_footprints:SOD_123F, symbol UNITED_DIODES_DATA_BASE:D_US1DWF
- removed D4: 100.0 V, diode_footprints:PowerDI_123, symbol UNITED_DIODES_DATA_BASE:D_DFLS1200-7
- removed D5: 62.0 V, diode_footprints:SOD_123, symbol UNITED_DIODES_DATA_BASE:D_MMSZ5265BT1G
- removed JP1, JP2: SolderJumper_2_Bridged, solder_jumper_footprints:SolderJumper-2_P1.3mm_Bridged_RoundedPad1.0x1.5mm, symbol UNITED_SOLDER_JUMPERS:SolderJumper_2_Bridged
- removed JP3: SolderJumper_3_Open, solder_jumper_footprints:SolderJumper-3_P1.3mm_Open_RoundedPad1.0x1.5mm_NumberLabels, symbol UNITED_SOLDER_JUMPERS:SolderJumper_3_Open
- removed L1: 2.2 µH, inductor_footprints:74479276, symbol UNITED_INDUCTORS_DATA_BASE:L_74479276222
- removed L2: 100.0 µH, inductor_footprints:74404032, symbol INDUCTORS_74404032_DATA_BASE:L_74404032101
- removed L3, L4: 100.0 µH, inductor_footprints:XFL3012, symbol UNITED_INDUCTORS_DATA_BASE:L_XFL3012-104ME
- removed R1, R2: 3.3 kΩ, resistor_footprints:R_0402_1005Metric, symbol RESISTORS_ERJ-2RKF_DATA_BASE:R_ERJ-2RKF3301X
- removed R10: 3.48 MΩ, resistor_footprints:R_0402_1005Metric, symbol UNITED_RESISTORS_DATA_BASE:R_RC0402FR-073M48L
- removed R11: 10 kΩ, resistor_footprints:R_0402_1005Metric, symbol UNITED_RESISTORS_DATA_BASE:R_ERJ-2RKF1002X
- removed R12, R23: 100 kΩ, resistor_footprints:R_0402_1005Metric, symbol UNITED_RESISTORS_DATA_BASE:R_ERJ-2GEJ104X
- removed R13: 604 kΩ, resistor_footprints:R_0402_1005Metric, symbol RESISTORS_ERJ-2RKF_DATA_BASE:R_ERJ-2RKF6043X
- removed R14: 2.2 MΩ, resistor_footprints:R_0402_1005Metric, symbol RESISTORS_RC0402FR-07_DATA_BASE:R_RC0402FR-072M2L
- removed R15: 150 kΩ, resistor_footprints:R_0402_1005Metric, symbol RESISTORS_ERJ-2RKF_DATA_BASE:R_ERJ-2RKF1503X
- removed R16: 30 kΩ, resistor_footprints:R_0402_1005Metric, symbol RESISTORS_ERJ-2RKF_DATA_BASE:R_ERJ-2RKF3002X
- removed R17: 470 kΩ, resistor_footprints:R_0402_1005Metric, symbol RESISTORS_RC0402FR-07_DATA_BASE:R_RC0402FR-07470KL
- removed R18: 40.2 kΩ, resistor_footprints:R_0402_1005Metric, symbol RESISTORS_ERJ-2RKF_DATA_BASE:R_ERJ-2RKF4022X
- removed R19: 3.32 MΩ, resistor_footprints:R_0402_1005Metric, symbol RESISTORS_RC0402FR-07_DATA_BASE:R_RC0402FR-073M32L
- removed R20: 294 kΩ, resistor_footprints:R_0402_1005Metric, symbol RESISTORS_ERJ-2RKF_DATA_BASE:R_ERJ-2RKF2943X
- removed R21, R22, R24, R25, R4: 1 kΩ, resistor_footprints:R_0402_1005Metric, symbol UNITED_RESISTORS_DATA_BASE:R_ERJ-2RKF1001X
- removed R3: 120 kΩ, resistor_footprints:R_0402_1005Metric, symbol UNITED_RESISTORS_DATA_BASE:R_ERJ-2RKF1203X
- removed R5: 9.76 kΩ, resistor_footprints:R_0402_1005Metric, symbol RESISTORS_ERJ-2RKF_DATA_BASE:R_ERJ-2RKF9761X
- removed R6: 121 kΩ, resistor_footprints:R_0402_1005Metric, symbol UNITED_RESISTORS_DATA_BASE:R_ERJ-2RKF1213X
- removed R7: 2.15 MΩ, resistor_footprints:R_0402_1005Metric, symbol UNITED_RESISTORS_DATA_BASE:R_RC0402FR-072M15L
- removed R8: 150 kΩ, resistor_footprints:R_0402_1005Metric, symbol RESISTORS_ERJ-2GEJ_DATA_BASE:R_ERJ-2GEJ154X
- removed R9: 15 kΩ, resistor_footprints:R_0402_1005Metric, symbol RESISTORS_ERJ-2RKF_DATA_BASE:R_ERJ-2RKF1502X
- removed T1: ZA9644-AED, transformer_footprints:ZA9644, symbol UNITED_TRANSFORMERS_DATA_BASE:T_ZA9644-AED
- removed TP1, TP10, TP11, TP12, TP13, TP14, TP15, TP16, TP17, TP18, TP19, TP2, TP20, TP21, TP22, TP23, TP25, TP26, TP28, TP29, TP3, TP30, TP31, TP32, TP33, TP34, TP35, TP36, TP37, TP38, TP39, TP4, TP40, TP41, TP42, TP43, TP44, TP45, TP46, TP47, TP48, TP49, TP5, TP50, TP51, TP52, TP56, TP57, TP6, TP7, TP8, TP9: TestPoint, test_point_footprints:TestPoint_THTPad_Castelated, symbol UNITED_TEST_POINTS:TestPoint_Castelated_v2
- removed TP24, TP27: TestPoint, test_point_footprints:TestPoint_THTPad_Castelated, symbol UNITED_TEST_POINTS:TestPoint_Castelated
- removed U1: MAX17227JATA+, analog_devices_footprints:21-0168_T822&plus_3C_ADI, symbol UNITED_IC_ADI:U_MAX17227JATA+
- removed U2: MAX17614ATP+, analog_devices_footprints:21-100172_T2044&plus_4C_MXM_ADI, symbol UNITED_IC_ADI:U_MAX17614ATP+
- removed U3: MAX17570FATA+, analog_devices_footprints:21-100514_T822C&plus_6C_ADI, symbol UNITED_IC_ADI:U_MAX17570FATA+
- removed U4: ADP1031ACPZ-3-R7, analog_devices_footprints:CP-41-1_ADI, symbol UNITED_IC_ADI:U_ADP1031ACPZ-3-R7
- removed U5, U6: ADUM340E0BRQZ, analog_devices_footprints:RQ-16_ADI, symbol UNITED_IC_ADI:U_ADUM340E0BRQZ
- removed U7: ADUM1252AUA+, analog_devices_footprints:21-0036_ADI, symbol UNITED_IC_ADI:U_ADUM1252AUA+
Connections:
- net DO_VDD: now also J4.1; no longer J4.2
- net GNDA: now also J4.2; no longer J4.1
- no-connect marks 9 -> 0
Other:
- added sheet Power_Supply_and_Digital_Interface (Power_Supply_and_Digital_Interface.kicad_sch)
- moved on the sheet: J1, J2, J3, J4

Commit message: backup
Parts:
- added MB4, MB6: mouse-bite-50mil-200mil, mouse_bite_footprints:mouse-bite-50mil-200mil, symbol UNITED_MOUSE_BITES_DATA_BASE:mouse-bite-50mil-200mil
Changed lines of the file:
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@@
+	)
+	(symbol
+		(lib_id "UNITED_MOUSE_BITES_DATA_BASE:mouse-bite-50mil-200mil")
+		(at 304.8 86.36 0)
+		(mirror y)
+		(unit 1)
+		(exclude_from_sim no)
+		(in_bom yes)
+		(on_board yes)
+		(dnp no)
+		(fields_autoplaced yes)
+		(property "Reference" "MB6"
+			(at 304.8 78.74 0)
+			(effects
+				(font
+					(size 1.27 1.27)
+				)
+				(justify left)
+				(hide yes)
+			)
+		)
+		(property "Value" "mouse-bite-50mil-200mil"
+			(at 304.8 93.98 0)
+			(effects
+				(font
+					(size 1.27 1.27)
+				)
+				(justify left)
+				(hide yes)
+			)
+		)
+		(property "Footprint" "mouse_bite_footprints:mouse-bite-50mil-200mil"
+			(at 304.8 91.44 0)
+			(effects
+				(font
+					(size 1.27 1.27)
+				)
+				(justify left)
+				(hide yes)
+			)
+		)
+		(property "Datasheet" ""
+			(at 304.8 86.36 0)
+			(effects
+				(font
+					(size 1.27 1.27)
+				)
+				(hide yes)
+			)
+		)
+		(property "Description" ""
+			(at 304.8 86.36 0)
+			(effects
+				(font
+					(size 1.27 1.27)
+				)
+				(hide yes)
+			)
+		)
+		(instances
+			(project "ad74416h_power_interface_module"
+				(path "/77c31fce-5dda-4017-bb4a-d31be1dfb2ec"
+					(reference "MB6")
+					(unit 1)
+				)
+			)
+		)
+	)
+	(symbol
+		(lib_id "UNITED_MOUSE_BITES_DATA_BASE:mouse-bite-50mil-200mil")
+		(at 101.6 81.28 0)
+		(unit 1)
+		(exclude_from_sim no)
+		(in_bom yes)
+		(on_board yes)
+		(dnp no)
+		(fields_autoplaced yes)
+		(property "Reference" "MB4"
+			(at 101.6 73.66 0)
+			(effects
+				(font
+					(size 1.27 1.27)
+				)
+				(justify left)
+				(hide yes)
+			)
+		)
+		(property "Value" "mouse-bite-50mil-200mil"
+			(at 101.6 88.9 0)
+			(effects
+				(font
+					(size 1.27 1.27)
+				)
+				(justify left)
+				(hide yes)
+			)
+		)
+		(property "Footprint" "mouse_bite_footprints:mouse-bite-50mil-200mil"
+			(at 101.6 86.36 0)
+			(effects
+				(font
+					(size 1.27 1.27)
+				)
+				(justify left)
+				(hide yes)
+			)
+		)
+		(property "Datasheet" ""
+			(at 101.6 81.28 0)
+			(effects
+				(font
+					(size 1.27 1.27)
+				)
+				(hide yes)
+			)
+		)
+		(property "Description" ""
+			(at 101.6 81.28 0)
+			(effects
+				(font
+					(size 1.27 1.27)
+				)
+				(hide yes)
+			)
+		)
+		(instances
+			(project "ad74416h_power_interface_module"
+				(path "/77c31fce-5dda-4017-bb4a-d31be1dfb2ec"
+					(reference "MB4")
+					(unit 1)
+				)
+			)
+		)
 	)
 	(symbol

Commit message: backup
Parts:
- added J5, J6: FW-06-03-G-D-085-155, connector_footprints:FW-06-03-G-D-085-155, symbol CONNECTORS_FW-xx-03-G-D-085-155_DATA_BASE:J_FW-06-03-G-D-085-155
- added TP53, TP54, TP55, TP58, TP59, TP60, TP63, TP64, TP67, TP68, TP69, TP70: TestPoint, test_point_footprints:TestPoint_THTPad_Castelated, symbol UNITED_TEST_POINTS:TestPoint_Castelated_v2
- MB1, MB3: value mouse-bite-50mil-200mil -> mouse-bite-50mil-300mil; footprint mouse_bite_footprints:mouse-bite-50mil-200mil -> mouse_bite_footprints:mouse-bite-50mil-300mil; symbol UNITED_MOUSE_BITES_DATA_BASE:mouse-bite-50mil-200mil -> UNITED_MOUSE_BITES_DATA_BASE:mouse-bite-50mil-300mil
- MB4, MB6: value mouse-bite-50mil-200mil -> mouse-bite-50mil-400mil; footprint mouse_bite_footprints:mouse-bite-50mil-200mil -> mouse_bite_footprints:mouse-bite-50mil-400mil; symbol UNITED_MOUSE_BITES_DATA_BASE:mouse-bite-50mil-200mil -> UNITED_MOUSE_BITES_DATA_BASE:mouse-bite-50mil-400mil
Connections:
- net DO_VDD: now also J6.10, J6.11, J6.12, J6.7, J6.8, J6.9, TP53.1, TP69.1, TP70.1
- net GND: now also J5.10, J5.11, J5.12, J5.7, J5.8, J5.9, TP55.1, TP60.1, TP63.1
- net GNDA: now also J6.1, J6.2, J6.3, J6.4, J6.5, J6.6, TP54.1, TP67.1, TP68.1
- net VINP: now also J5.1, J5.2, J5.3, J5.4, J5.5, J5.6, TP58.1, TP59.1, TP64.1

Commit message: backup
Parts:
- removed TP63, TP64, TP68, TP70: TestPoint, test_point_footprints:TestPoint_THTPad_Castelated, symbol UNITED_TEST_POINTS:TestPoint_Castelated_v2
- J3: renamed from J5; value FW-06-03-G-D-085-155 -> FW-04-03-G-D-085-155; footprint connector_footprints:FW-06-03-G-D-085-155 -> connector_footprints:FW-04-03-G-D-085-155; symbol CONNECTORS_FW-xx-03-G-D-085-155_DATA_BASE:J_FW-06-03-G-D-085-155 -> CONNECTORS_FW-xx-03-G-D-085-155_DATA_BASE:J_FW-04-03-G-D-085-155; MPN FW-06-03-G-D-085-155 -> FW-04-03-G-D-085-155; Pin Count 6 -> 4; Symbol Name J_FW-06-03-G-D-085-155 -> J_FW-04-03-G-D-085-155; Trustedparts Search https://www.trustedparts.com/en/search/FW-06-03-G-D-085-155 -> https://www.trustedparts.com/en/search/FW-04-03-G-D-085-155
- J5: renamed from J6; value FW-06-03-G-D-085-155 -> FW-04-03-G-D-085-155; footprint connector_footprints:FW-06-03-G-D-085-155 -> connector_footprints:FW-04-03-G-D-085-155; symbol CONNECTORS_FW-xx-03-G-D-085-155_DATA_BASE:J_FW-06-03-G-D-085-155 -> CONNECTORS_FW-xx-03-G-D-085-155_DATA_BASE:J_FW-04-03-G-D-085-155; MPN FW-06-03-G-D-085-155 -> FW-04-03-G-D-085-155; Pin Count 6 -> 4; Symbol Name J_FW-06-03-G-D-085-155 -> J_FW-04-03-G-D-085-155; Trustedparts Search https://www.trustedparts.com/en/search/FW-06-03-G-D-085-155 -> https://www.trustedparts.com/en/search/FW-04-03-G-D-085-155
- MB2: renamed from MB4; value mouse-bite-50mil-400mil -> mouse-bite-50mil-300mil; footprint mouse_bite_footprints:mouse-bite-50mil-400mil -> mouse_bite_footprints:mouse-bite-50mil-300mil; symbol UNITED_MOUSE_BITES_DATA_BASE:mouse-bite-50mil-400mil -> UNITED_MOUSE_BITES_DATA_BASE:mouse-bite-50mil-300mil
- MB4: renamed from MB6; value mouse-bite-50mil-400mil -> mouse-bite-50mil-300mil; footprint mouse_bite_footprints:mouse-bite-50mil-400mil -> mouse_bite_footprints:mouse-bite-50mil-300mil; symbol UNITED_MOUSE_BITES_DATA_BASE:mouse-bite-50mil-400mil -> UNITED_MOUSE_BITES_DATA_BASE:mouse-bite-50mil-300mil
- renumbered J3 to J4, J4 to J6, MB5 to MB1, MB2 to MB3, MB1 to MB5, MB3 to MB6, TP59 to TP34, TP58 to TP35, TP55 to TP36, TP60 to TP37, TP67 to TP55, TP54 to TP56, TP53 to TP57, TP69 to TP58
Connections:
- net DO_VDD: now also J5.5, J5.6; no longer J5.10, J5.11, J5.12, J5.9
- net GND: now also J3.5, J3.6; no longer J3.10, J3.11, J3.12, J3.9
- net GNDA: no longer J5.5, J5.6
- net VINP: no longer J3.5, J3.6
Other:
- moved on the sheet: TP34, TP35, TP36, TP37, TP55, TP56, TP57, TP58

Commit message: backup
Parts:
- removed MB5, MB6: mouse-bite-50mil-300mil, mouse_bite_footprints:mouse-bite-50mil-300mil, symbol UNITED_MOUSE_BITES_DATA_BASE:mouse-bite-50mil-300mil
- J1: value FW-33-03-G-D-085-155 -> FW-33-03-G-D-150-160; footprint connector_footprints:FW-33-03-G-D-085-155 -> connector_footprints:FW-33-03-G-D-150-160; symbol CONNECTORS_FW-xx-03-G-D-085-155_DATA_BASE:J_FW-33-03-G-D-085-155 -> CONNECTORS_FW-xx-03-G-D-150-160_DATA_BASE:J_FW-33-03-G-D-150-160; MPN FW-33-03-G-D-085-155 -> FW-33-03-G-D-150-160; Series FW-xx-03-G-D-085-155 -> FW-xx-03-G-D-150-160; Symbol Name J_FW-33-03-G-D-085-155 -> J_FW-33-03-G-D-150-160; Trustedparts Search https://www.trustedparts.com/en/search/FW-33-03-G-D-085-155 -> https://www.trustedparts.com/en/search/FW-33-03-G-D-150-160
Changed lines of the file:
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@@
 	)
 	(symbol
-		(lib_id "CONNECTORS_FW-xx-03-G-D-085-155_DATA_BASE:J_FW-33-03-G-D-085-155")
+		(lib_id "CONNECTORS_FW-xx-03-G-D-150-160_DATA_BASE:J_FW-33-03-G-D-150-160")
 		(at 304.8 160.02 0)
 		(unit 1)
@@
 			)
 		)
-		(property "Value" "FW-33-03-G-D-085-155"
+		(property "Value" "FW-33-03-G-D-150-160"
 			(at 304.8 114.3 0)
 			(effects
@@
 			)
 		)
-		(property "Footprint" "connector_footprints:FW-33-03-G-D-085-155"
+		(property "Footprint" "connector_footprints:FW-33-03-G-D-150-160"
 			(at 309.88 207.01 0)
 			(show_name yes)
@@
 			)
 		)
-		(property "Datasheet" "https://suddendocs.samtec.com/catalog_english/fw_sm.pdf?_gl=1*1xtxv9c*_gcl_au*MTM0MTYyNTQ5MS4xNzM2MDk5MTUz*_ga*MTYxNDYyMTQ0Mi4xNzM2MDk5MTUz*_ga_3KFNZC07WW*MTczODE2NTI0NS4zMi4xLjE3MzgxNjU1NjMuNjAuMC4w"
+		(property "Datasheet" "https://suddendocs.samtec.com/catalog_english/fw_sm.pdf?_gl=1*696njn*_gcl_au*OTQ3NjE2MTIwLjE3NTQ5MDMyODE.*_ga*NzIxODQzNjU3LjE3NTQ5MDMyODI.*_ga_3KFNZC07WW*czE3NTk0NzU3MTckbzkkZzEkdDE3NTk0Nzk3ODIkajYwJGwwJGgw"
 			(at 309.88 209.55 0)
 			(show_name yes)
@@
 			)
 		)
-		(property "Description" "Samtec FW-xx-03-G-D-085-155 series,  33 positions connector,  1.27 mm pitch,  Black,  Vertical mounting,  5.2 A,  300 V,  Surface Mount,  Gold plated"
+		(property "Description" "Samtec FW-xx-03-G-D-150-160 series,  33 positions connector,  1.27 mm pitch,  Black,  Vertical mounting,  5.2 A,  300 V,  Surface Mount,  Gold plated"
 			(at 309.88 212.09 0)
 			(show_name yes)
@@
 			)
 		)
-		(property "MPN" "FW-33-03-G-D-085-155"
+		(property "MPN" "FW-33-03-G-D-150-160"
 			(at 309.88 222.25 0)
 			(show_name yes)
@@
 			)
 		)
-		(property "Series" "FW-xx-03-G-D-085-155"
+		(property "Series" "FW-xx-03-G-D-150-160"
 			(at 309.88 240.03 0)
 			(show_name yes)
@@
 			)
 		)
-		(property "Symbol Name" "J_FW-33-03-G-D-085-155"
+		(property "Symbol Name" "J_FW-33-03-G-D-150-160"
 			(at 309.88 242.57 0)
 			(show_name yes)
@@
 			)
 		)
-		(property "Trustedparts Search" "https://www.trustedparts.com/en/search/FW-33-03-G-D-085-155"
+		(property "Trustedparts Search" "https://www.trustedparts.com/en/search/FW-33-03-G-D-150-160"
 			(at 309.88 245.11 0)
 			(show_name yes)
@@
 	)
 	(symbol
-		(lib_id "UNITED_MOUSE_BITES_DATA_BASE:mouse-bite-50mil-300mil")
-		(at 101.6 106.68 0)
-		(unit 1)
-		(exclude_from_sim no)
-		(in_bom yes)
-		(on_board yes)
-		(dnp no)
-		(fields_autoplaced yes)
-		(property "Reference" "MB5"
-			(at 101.6 99.06 0)
-			(effects
-				(font
-					(size 1.27 1.27)
-				)
-				(justify left)
-				(hide yes)
-			)
-		)
-		(property "Value" "mouse-bite-50mil-300mil"
-			(at 101.6 114.3 0)
-			(effects
-				(font
-					(size 1.27 1.27)
-				)
-				(justify left)
-				(hide yes)
-			)
-		)
-		(property "Footprint" "mouse_bite_footprints:mouse-bite-50mil-300mil"
-			(at 101.6 111.76 0)
-			(effects
-				(font
-					(size 1.27 1.27)
-				)
-				(justify left)
-				(hide yes)
-			)
-		)
-		(property "Datasheet" ""
-			(at 101.6 106.68 0)
-			(effects
-				(font
-					(size 1.27 1.27)
-				)
-				(hide yes)
-			)
-		)
-		(property "Description" ""
-			(at 101.6 106.68 0)
-			(effects
-				(font
-					(size 1.27 1.27)
-				)
-				(hide yes)
-			)
-		)
-		(instances
-			(project ""
-				(path "/77c31fce-5dda-4017-bb4a-d31be1dfb2ec"
-					(reference "MB5")
-					(unit 1)
-				)
-			)
-		)
-	)
-	(symbol
 		(lib_id "CONNECTORS_TBP02R1-381_DATA_BASE:J_TBP02R1-381-02BE")
 		(at 101.6 95.25 180)
@@
 					(unit 1)
 				)
-			)
-		)
-	)
-	(symbol
-		(lib_id "UNITED_MOUSE_BITES_DATA_BASE:mouse-bite-50mil-300mil")
-		(at 304.8 106.68 0)
-		(mirror y)
-		(unit 1)
-		(exclude_from_sim no)
-		(in_bom yes)
-		(on_board yes)
-		(dnp no)
-		(fields_autoplaced yes)
-		(property "Reference" "MB6"
-			(at 304.8 99.06 0)
-			(effects
-				(font
-					(size 1.27 1.27)
-				)
-				(justify left)
-				(hide yes)
-			)
-		)
-		(property "Value" "mouse-bite-50mil-300mil"
-			(at 304.8 114.3 0)
-			(effects
-				(font
-					(size 1.27 1.27)
-				)
-				(justify left)
-				(hide yes)
-			)
-		)
-		(property "Footprint" "mouse_bite_footprints:mouse-bite-50mil-300mil"
-			(at 304.8 111.76 0)
-			(effects
-				(font
-					(size 1.27 1.27)
-				)
-				(justify left)
-				(hide yes)
-			)
-		)
-		(property "Datasheet" ""
-			(at 304.8 106.68 0)
-			(effects
-				(font
-					(size 1.27 1.27)
-				)
-				(hide yes)
-			)
-		)
-		(property "Description" ""
-			(at 304.8 106.68 0)
-			(effects
-				(font
-					(size 1.27 1.27)
-				)
-				(hide yes)
-			)
-		)
-		(instances
-			(project "ad74416h_power_interface_module"
-				(path "/77c31fce-5dda-4017-bb4a-d31be1dfb2ec"
-					(reference "MB6")
-					(unit 1)
-				)
