File: ad74416h_power_interface_module/ad74416h_power_interface_module.kicad_sch (KiCad schematic)
At the start: 18 parts, among them J1 FW-33-03-G-D-150-160, J2 TBP02R1-381-02BE, J3 FW-04-03-G-D-085-155, J4 FW-17-03-G-D-085-155, J5 FW-04-03-G-D-085-155, J6 TBP02R1-381-02BE

Commit message: backup
Parts:
- J3: value FW-04-03-G-D-085-155 -> FW-04-05-G-D-470-160; footprint connector_footprints:FW-04-03-G-D-085-155 -> connector_footprints:FW-04-05-G-D-470-160; symbol CONNECTORS_FW-xx-03-G-D-085-155_DATA_BASE:J_FW-04-03-G-D-085-155 -> CONNECTORS_FW-xx-05-G-D-470-160_DATA_BASE:J_FW-04-05-G-D-470-160; MPN FW-04-03-G-D-085-155 -> FW-04-05-G-D-470-160; Series FW-xx-03-G-D-085-155 -> FW-xx-05-G-D-470-160; Symbol Name J_FW-04-03-G-D-085-155 -> J_FW-04-05-G-D-470-160; Trustedparts Search https://www.trustedparts.com/en/search/FW-04-03-G-D-085-155 -> https://www.trustedparts.com/en/search/FW-04-05-G-D-470-160
- J4: value FW-17-03-G-D-085-155 -> CLP-117-02-G-D-BE; footprint connector_footprints:FW-17-03-G-D-085-155 -> connector_footprints:CLP-117-02-G-D-BE; symbol CONNECTORS_FW-xx-03-G-D-085-155_DATA_BASE:J_FW-17-03-G-D-085-155 -> CONNECTORS_CLP-1xx-02-G-D-BE_DATA_BASE:J_CLP-117-02-G-D-BE; Contact Plating Gold -> Tin; MPN FW-17-03-G-D-085-155 -> CLP-117-02-G-D-BE; Series FW-xx-03-G-D-085-155 -> CLP-1xx-02-G-D-BE; Symbol Name J_FW-17-03-G-D-085-155 -> J_CLP-117-02-G-D-BE; Trustedparts Search https://www.trustedparts.com/en/search/FW-17-03-G-D-085-155 -> https://www.trustedparts.com/en/search/CLP-117-02-G-D-BE
- J5: value FW-04-03-G-D-085-155 -> FW-04-05-F-D-248-160; footprint connector_footprints:FW-04-03-G-D-085-155 -> connector_footprints:FW-04-05-F-D-248-160; symbol CONNECTORS_FW-xx-03-G-D-085-155_DATA_BASE:J_FW-04-03-G-D-085-155 -> CONNECTORS_FW-xx-05-F-D-248-160_DATA_BASE:J_FW-04-05-F-D-248-160; MPN FW-04-03-G-D-085-155 -> FW-04-05-F-D-248-160; Series FW-xx-03-G-D-085-155 -> FW-xx-05-F-D-248-160; Symbol Name J_FW-04-03-G-D-085-155 -> J_FW-04-05-F-D-248-160; Trustedparts Search https://www.trustedparts.com/en/search/FW-04-03-G-D-085-155 -> https://www.trustedparts.com/en/search/FW-04-05-F-D-248-160
Changed lines of the file:
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@@
 	)
 	(symbol
-		(lib_id "CONNECTORS_FW-xx-03-G-D-085-155_DATA_BASE:J_FW-17-03-G-D-085-155")
+		(lib_id "CONNECTORS_CLP-1xx-02-G-D-BE_DATA_BASE:J_CLP-117-02-G-D-BE")
 		(at 101.6 139.7 0)
 		(unit 1)
@@
 			)
 		)
-		(property "Value" "FW-17-03-G-D-085-155"
+		(property "Value" "CLP-117-02-G-D-BE"
 			(at 101.6 114.3 0)
 			(effects
@@
 			)
 		)
-		(property "Footprint" "connector_footprints:FW-17-03-G-D-085-155"
+		(property "Footprint" "connector_footprints:CLP-117-02-G-D-BE"
 			(at 106.68 166.37 0)
 			(show_name yes)
@@
 			)
 		)
-		(property "Datasheet" "https://suddendocs.samtec.com/catalog_english/fw_sm.pdf?_gl=1*1xtxv9c*_gcl_au*MTM0MTYyNTQ5MS4xNzM2MDk5MTUz*_ga*MTYxNDYyMTQ0Mi4xNzM2MDk5MTUz*_ga_3KFNZC07WW*MTczODE2NTI0NS4zMi4xLjE3MzgxNjU1NjMuNjAuMC4w"
+		(property "Datasheet" "https://suddendocs.samtec.com/catalog_english/clp_sm.pdf?_gl=1*1y4jlr9*_gcl_au*MTM0MTYyNTQ5MS4xNzM2MDk5MTUz*_ga*MTYxNDYyMTQ0Mi4xNzM2MDk5MTUz*_ga_3KFNZC07WW*MTczNjY4MDQ4OS4xNS4xLjE3MzY2ODEzNzcuNjAuMC4w"
 			(at 106.68 168.91 0)
 			(show_name yes)
@@
 			)
 		)
-		(property "Description" "Samtec FW-xx-03-G-D-085-155 series,  17 positions connector,  1.27 mm pitch,  Black,  Vertical mounting,  5.2 A,  300 V,  Surface Mount,  Gold plated"
+		(property "Description" "Samtec CLP-1xx-02-G-D-BE series,  17 positions connector,  1.27 mm pitch,  Black,  Vertical mounting,  5.2 A,  300 V,  Surface Mount,  Tin plated"
 			(at 106.68 171.45 0)
 			(show_name yes)
@@
 			)
 		)
-		(property "Contact Plating" "Gold"
+		(property "Contact Plating" "Tin"
 			(at 106.68 176.53 0)
 			(show_name yes)
@@
 			)
 		)
-		(property "MPN" "FW-17-03-G-D-085-155"
+		(property "MPN" "CLP-117-02-G-D-BE"
 			(at 106.68 181.61 0)
 			(show_name yes)
@@
 			)
 		)
-		(property "Series" "FW-xx-03-G-D-085-155"
+		(property "Series" "CLP-1xx-02-G-D-BE"
 			(at 106.68 199.39 0)
 			(show_name yes)
@@
 			)
 		)
-		(property "Symbol Name" "J_FW-17-03-G-D-085-155"
+		(property "Symbol Name" "J_CLP-117-02-G-D-BE"
 			(at 106.68 201.93 0)
 			(show_name yes)
@@
 			)
 		)
-		(property "Trustedparts Search" "https://www.trustedparts.com/en/search/FW-17-03-G-D-085-155"
+		(property "Trustedparts Search" "https://www.trustedparts.com/en/search/CLP-117-02-G-D-BE"
 			(at 106.68 204.47 0)
 			(show_name yes)
@@
 	)
 	(symbol
-		(lib_id "CONNECTORS_FW-xx-03-G-D-085-155_DATA_BASE:J_FW-04-03-G-D-085-155")
+		(lib_id "CONNECTORS_FW-xx-05-G-D-470-160_DATA_BASE:J_FW-04-05-G-D-470-160")
 		(at 101.6 72.39 0)
 		(unit 1)
@@
 			)
 		)
-		(property "Value" "FW-04-03-G-D-085-155"
+		(property "Value" "FW-04-05-G-D-470-160"
 			(at 101.6 63.5 0)
 			(effects
@@
 			)
 		)
-		(property "Footprint" "connector_footprints:FW-04-03-G-D-085-155"
+		(property "Footprint" "connector_footprints:FW-04-05-G-D-470-160"
 			(at 106.68 82.55 0)
 			(show_name yes)
@@
 			)
 		)
-		(property "Datasheet" "https://suddendocs.samtec.com/catalog_english/fw_sm.pdf?_gl=1*1xtxv9c*_gcl_au*MTM0MTYyNTQ5MS4xNzM2MDk5MTUz*_ga*MTYxNDYyMTQ0Mi4xNzM2MDk5MTUz*_ga_3KFNZC07WW*MTczODE2NTI0NS4zMi4xLjE3MzgxNjU1NjMuNjAuMC4w"
+		(property "Datasheet" "https://suddendocs.samtec.com/catalog_english/fw_sm.pdf?_gl=1*dqfgvk*_gcl_au*OTQ3NjE2MTIwLjE3NTQ5MDMyODE.*_ga*NzIxODQzNjU3LjE3NTQ5MDMyODI.*_ga_3KFNZC07WW*czE3NTk3NjQxNTMkbzEyJGcwJHQxNzU5NzY1NzUzJGo2MCRsMCRoMA.."
 			(at 106.68 85.09 0)
 			(show_name yes)
@@
 			)
 		)
-		(property "Description" "Samtec FW-xx-03-G-D-085-155 series,  4 positions connector,  1.27 mm pitch,  Black,  Vertical mounting,  5.2 A,  300 V,  Surface Mount,  Gold plated"
+		(property "Description" "Samtec FW-xx-05-G-D-470-160 series,  4 positions connector,  1.27 mm pitch,  Black,  Vertical mounting,  5.2 A,  300 V,  Surface Mount,  Gold plated"
 			(at 106.68 87.63 0)
 			(show_name yes)
@@
 			)
 		)
-		(property "MPN" "FW-04-03-G-D-085-155"
+		(property "MPN" "FW-04-05-G-D-470-160"
 			(at 106.68 97.79 0)
 			(show_name yes)
@@
 			)
 		)
-		(property "Series" "FW-xx-03-G-D-085-155"
+		(property "Series" "FW-xx-05-G-D-470-160"
 			(at 106.68 115.57 0)
 			(show_name yes)
@@
 			)
 		)
-		(property "Symbol Name" "J_FW-04-03-G-D-085-155"
+		(property "Symbol Name" "J_FW-04-05-G-D-470-160"
 			(at 106.68 118.11 0)
 			(show_name yes)
@@
 			)
 		)
-		(property "Trustedparts Search" "https://www.trustedparts.com/en/search/FW-04-03-G-D-085-155"
+		(property "Trustedparts Search" "https://www.trustedparts.com/en/search/FW-04-05-G-D-470-160"
 			(at 106.68 120.65 0)
 			(show_name yes)
@@
 	)
 	(symbol
-		(lib_id "CONNECTORS_FW-xx-03-G-D-085-155_DATA_BASE:J_FW-04-03-G-D-085-155")
+		(lib_id "CONNECTORS_FW-xx-05-F-D-248-160_DATA_BASE:J_FW-04-05-F-D-248-160")
 		(at 304.8 72.39 0)
 		(mirror x)
@@
 			)
 		)
-		(property "Value" "FW-04-03-G-D-085-155"
+		(property "Value" "FW-04-05-F-D-248-160"
 			(at 304.8 63.5 0)
 			(effects
@@
 			)
 		)
-		(property "Footprint" "connector_footprints:FW-04-03-G-D-085-155"
+		(property "Footprint" "connector_footprints:FW-04-05-F-D-248-160"
 			(at 309.88 62.23 0)
 			(show_name yes)
@@
 			)
 		)
-		(property "Datasheet" "https://suddendocs.samtec.com/catalog_english/fw_sm.pdf?_gl=1*1xtxv9c*_gcl_au*MTM0MTYyNTQ5MS4xNzM2MDk5MTUz*_ga*MTYxNDYyMTQ0Mi4xNzM2MDk5MTUz*_ga_3KFNZC07WW*MTczODE2NTI0NS4zMi4xLjE3MzgxNjU1NjMuNjAuMC4w"
+		(property "Datasheet" "https://suddendocs.samtec.com/catalog_english/fw_sm.pdf?_gl=1*1mheflh*_gcl_au*OTQ3NjE2MTIwLjE3NTQ5MDMyODE.*_ga*NzIxODQzNjU3LjE3NTQ5MDMyODI.*_ga_3KFNZC07WW*czE3NTk0MTUxODQkbzckZzEkdDE3NTk0MTc0NDAkajYwJGwwJGgw"
 			(at 309.88 59.69 0)
 			(show_name yes)
@@
 			)
 		)
-		(property "Description" "Samtec FW-xx-03-G-D-085-155 series,  4 positions connector,  1.27 mm pitch,  Black,  Vertical mounting,  5.2 A,  300 V,  Surface Mount,  Gold plated"
+		(property "Description" "Samtec FW-xx-05-F-D-248-160 series,  4 positions connector,  1.27 mm pitch,  Black,  Vertical mounting,  5.2 A,  300 V,  Surface Mount,  Gold plated"
 			(at 309.88 57.15 0)
 			(show_name yes)
@@
 			)
 		)
-		(property "MPN" "FW-04-03-G-D-085-155"
+		(property "MPN" "FW-04-05-F-D-248-160"
 			(at 309.88 46.99 0)
 			(show_name yes)
@@
 			)
 		)
-		(property "Series" "FW-xx-03-G-D-085-155"
+		(property "Series" "FW-xx-05-F-D-248-160"
 			(at 309.88 29.21 0)
 			(show_name yes)
@@
 			)
 		)
-		(property "Symbol Name" "J_FW-04-03-G-D-085-155"
+		(property "Symbol Name" "J_FW-04-05-F-D-248-160"
 			(at 309.88 26.67 0)
 			(show_name yes)
@@
 			)
 		)
-		(property "Trustedparts Search" "https://www.trustedparts.com/en/search/FW-04-03-G-D-085-155"
+		(property "Trustedparts Search" "https://www.trustedparts.com/en/search/FW-04-05-F-D-248-160"
 			(at 309.88 24.13 0)
 			(show_name yes)

Commit message: backup
Parts:
- J1: value FW-33-03-G-D-150-160 -> FTSH-133-04-L-DH; footprint connector_footprints:FW-33-03-G-D-150-160 -> connector_footprints:FTSH-133-04-L-DH; symbol CONNECTORS_FW-xx-03-G-D-150-160_DATA_BASE:J_FW-33-03-G-D-150-160 -> CONNECTORS_FTSH-1xx-04-L-DH_DATA_BASE:J_FTSH-133-04-L-DH; Contact Plating Gold -> Tin; MPN FW-33-03-G-D-150-160 -> FTSH-133-04-L-DH; Mounting Angle Vertical -> Horizontal; Series FW-xx-03-G-D-150-160 -> FTSH-1xx-04-L-DH; Symbol Name J_FW-33-03-G-D-150-160 -> J_FTSH-133-04-L-DH; Trustedparts Search https://www.trustedparts.com/en/search/FW-33-03-G-D-150-160 -> https://www.trustedparts.com/en/search/FTSH-133-04-L-DH
Changed lines of the file:
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@@
 	)
 	(symbol
-		(lib_id "CONNECTORS_FW-xx-03-G-D-150-160_DATA_BASE:J_FW-33-03-G-D-150-160")
+		(lib_id "CONNECTORS_FTSH-1xx-04-L-DH_DATA_BASE:J_FTSH-133-04-L-DH")
 		(at 304.8 160.02 0)
 		(unit 1)
@@
 			)
 		)
-		(property "Value" "FW-33-03-G-D-150-160"
+		(property "Value" "FTSH-133-04-L-DH"
 			(at 304.8 114.3 0)
 			(effects
@@
 			)
 		)
-		(property "Footprint" "connector_footprints:FW-33-03-G-D-150-160"
+		(property "Footprint" "connector_footprints:FTSH-133-04-L-DH"
 			(at 309.88 207.01 0)
 			(show_name yes)
@@
 			)
 		)
-		(property "Datasheet" "https://suddendocs.samtec.com/catalog_english/fw_sm.pdf?_gl=1*696njn*_gcl_au*OTQ3NjE2MTIwLjE3NTQ5MDMyODE.*_ga*NzIxODQzNjU3LjE3NTQ5MDMyODI.*_ga_3KFNZC07WW*czE3NTk0NzU3MTckbzkkZzEkdDE3NTk0Nzk3ODIkajYwJGwwJGgw"
+		(property "Datasheet" "https://suddendocs.samtec.com/catalog_english/ftsh_smt.pdf?_gl=1*uwyfuk*_gcl_au*OTQ3NjE2MTIwLjE3NTQ5MDMyODE.*_ga*NzIxODQzNjU3LjE3NTQ5MDMyODI.*_ga_3KFNZC07WW*czE3NTk5OTE3NDIkbzE1JGcxJHQxNzU5OTkxODU5JGo4JGwwJGgw"
 			(at 309.88 209.55 0)
 			(show_name yes)
@@
 			)
 		)
-		(property "Description" "Samtec FW-xx-03-G-D-150-160 series,  33 positions connector,  1.27 mm pitch,  Black,  Vertical mounting,  5.2 A,  300 V,  Surface Mount,  Gold plated"
+		(property "Description" "Samtec FTSH-1xx-04-L-DH series,  33 positions connector,  1.27 mm pitch,  Black,  Horizontal mounting,  5.2 A,  300 V,  Surface Mount,  Tin plated"
 			(at 309.88 212.09 0)
 			(show_name yes)
@@
 			)
 		)
-		(property "Contact Plating" "Gold"
+		(property "Contact Plating" "Tin"
 			(at 309.88 217.17 0)
 			(show_name yes)
@@
 			)
 		)
-		(property "MPN" "FW-33-03-G-D-150-160"
+		(property "MPN" "FTSH-133-04-L-DH"
 			(at 309.88 222.25 0)
 			(show_name yes)
@@
 			)
 		)
-		(property "Mounting Angle" "Vertical"
+		(property "Mounting Angle" "Horizontal"
 			(at 309.88 227.33 0)
 			(show_name yes)
@@
 			)
 		)
-		(property "Series" "FW-xx-03-G-D-150-160"
+		(property "Series" "FTSH-1xx-04-L-DH"
 			(at 309.88 240.03 0)
 			(show_name yes)
@@
 			)
 		)
-		(property "Symbol Name" "J_FW-33-03-G-D-150-160"
+		(property "Symbol Name" "J_FTSH-133-04-L-DH"
 			(at 309.88 242.57 0)
 			(show_name yes)
@@
 			)
 		)
-		(property "Trustedparts Search" "https://www.trustedparts.com/en/search/FW-33-03-G-D-150-160"
+		(property "Trustedparts Search" "https://www.trustedparts.com/en/search/FTSH-133-04-L-DH"
 			(at 309.88 245.11 0)
 			(show_name yes)

Commit message: backup
Parts:
- J1: value FTSH-133-04-L-DH -> CLP-133-02-G-D-BE; footprint connector_footprints:FTSH-133-04-L-DH -> connector_footprints:CLP-133-02-G-D-BE; symbol CONNECTORS_FTSH-1xx-04-L-DH_DATA_BASE:J_FTSH-133-04-L-DH -> CONNECTORS_CLP-1xx-02-G-D-BE_DATA_BASE:J_CLP-133-02-G-D-BE; MPN FTSH-133-04-L-DH -> CLP-133-02-G-D-BE; Mounting Angle Horizontal -> Vertical; Series FTSH-1xx-04-L-DH -> CLP-1xx-02-G-D-BE; Symbol Name J_FTSH-133-04-L-DH -> J_CLP-133-02-G-D-BE; Trustedparts Search https://www.trustedparts.com/en/search/FTSH-133-04-L-DH -> https://www.trustedparts.com/en/search/CLP-133-02-G-D-BE
Changed lines of the file:
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@@
 	)
 	(symbol
-		(lib_id "CONNECTORS_FTSH-1xx-04-L-DH_DATA_BASE:J_FTSH-133-04-L-DH")
+		(lib_id "CONNECTORS_CLP-1xx-02-G-D-BE_DATA_BASE:J_CLP-133-02-G-D-BE")
 		(at 304.8 160.02 0)
 		(unit 1)
@@
 			)
 		)
-		(property "Value" "FTSH-133-04-L-DH"
+		(property "Value" "CLP-133-02-G-D-BE"
 			(at 304.8 114.3 0)
 			(effects
@@
 			)
 		)
-		(property "Footprint" "connector_footprints:FTSH-133-04-L-DH"
+		(property "Footprint" "connector_footprints:CLP-133-02-G-D-BE"
 			(at 309.88 207.01 0)
 			(show_name yes)
@@
 			)
 		)
-		(property "Datasheet" "https://suddendocs.samtec.com/catalog_english/ftsh_smt.pdf?_gl=1*uwyfuk*_gcl_au*OTQ3NjE2MTIwLjE3NTQ5MDMyODE.*_ga*NzIxODQzNjU3LjE3NTQ5MDMyODI.*_ga_3KFNZC07WW*czE3NTk5OTE3NDIkbzE1JGcxJHQxNzU5OTkxODU5JGo4JGwwJGgw"
+		(property "Datasheet" "https://suddendocs.samtec.com/catalog_english/clp_sm.pdf?_gl=1*1y4jlr9*_gcl_au*MTM0MTYyNTQ5MS4xNzM2MDk5MTUz*_ga*MTYxNDYyMTQ0Mi4xNzM2MDk5MTUz*_ga_3KFNZC07WW*MTczNjY4MDQ4OS4xNS4xLjE3MzY2ODEzNzcuNjAuMC4w"
 			(at 309.88 209.55 0)
 			(show_name yes)
@@
 			)
 		)
-		(property "Description" "Samtec FTSH-1xx-04-L-DH series,  33 positions connector,  1.27 mm pitch,  Black,  Horizontal mounting,  5.2 A,  300 V,  Surface Mount,  Tin plated"
+		(property "Description" "Samtec CLP-1xx-02-G-D-BE series,  33 positions connector,  1.27 mm pitch,  Black,  Vertical mounting,  5.2 A,  300 V,  Surface Mount,  Tin plated"
 			(at 309.88 212.09 0)
 			(show_name yes)
@@
 			)
 		)
-		(property "MPN" "FTSH-133-04-L-DH"
+		(property "MPN" "CLP-133-02-G-D-BE"
 			(at 309.88 222.25 0)
 			(show_name yes)
@@
 			)
 		)
-		(property "Mounting Angle" "Horizontal"
+		(property "Mounting Angle" "Vertical"
 			(at 309.88 227.33 0)
 			(show_name yes)
@@
 			)
 		)
-		(property "Series" "FTSH-1xx-04-L-DH"
+		(property "Series" "CLP-1xx-02-G-D-BE"
 			(at 309.88 240.03 0)
 			(show_name yes)
@@
 			)
 		)
-		(property "Symbol Name" "J_FTSH-133-04-L-DH"
+		(property "Symbol Name" "J_CLP-133-02-G-D-BE"
 			(at 309.88 242.57 0)
 			(show_name yes)
@@
 			)
 		)
-		(property "Trustedparts Search" "https://www.trustedparts.com/en/search/FTSH-133-04-L-DH"
+		(property "Trustedparts Search" "https://www.trustedparts.com/en/search/CLP-133-02-G-D-BE"
 			(at 309.88 245.11 0)
 			(show_name yes)

Commit message: backup
Parts:
- added TP59, TP60: TestPoint, test_point_footprints:TestPoint_THTPad_Castelated, symbol UNITED_TEST_POINTS:TestPoint_Castelated_v2
- J1: value CLP-133-02-G-D-BE -> CLP-135-02-G-D-BE; footprint connector_footprints:CLP-133-02-G-D-BE -> connector_footprints:CLP-135-02-G-D-BE; symbol CONNECTORS_CLP-1xx-02-G-D-BE_DATA_BASE:J_CLP-133-02-G-D-BE -> CONNECTORS_CLP-1xx-02-G-D-BE_DATA_BASE:J_CLP-135-02-G-D-BE; MPN CLP-133-02-G-D-BE -> CLP-135-02-G-D-BE; Pin Count 33 -> 35; Symbol Name J_CLP-133-02-G-D-BE -> J_CLP-135-02-G-D-BE; Trustedparts Search https://www.trustedparts.com/en/search/CLP-133-02-G-D-BE -> https://www.trustedparts.com/en/search/CLP-135-02-G-D-BE
- MB1: value mouse-bite-50mil-1750mil -> mouse-bite-50mil-1850mil; footprint mouse_bite_footprints:mouse-bite-50mil-1750mil -> mouse_bite_footprints:mouse-bite-50mil-1850mil; symbol UNITED_MOUSE_BITES_DATA_BASE:mouse-bite-50mil-1750mil -> UNITED_MOUSE_BITES_DATA_BASE:mouse-bite-50mil-1850mil
Connections:
- net 14V5: now also J1.67, J1.68; no longer J1.63, J1.64
- net DO_VDD: now also J1.61, J1.62; no longer J1.57, J1.58
- net GNDA: now also J1.57, J1.58, J1.63, J1.64, J1.69, J1.70; no longer J1.53, J1.54, J1.55, J1.56, J1.61, J1.62
- no-connect marks 0 -> 4

Commit message: backup
Parts:
- added J10, J7: TBP02P1-381-02BE, terminal_block_footprints:TBP02P1-381-02BE, symbol TERMINAL_BLOCKS_TBP02P1-381_DATA_BASE:J_TBP02P1-381-02BE
